File: Project/HP2621.kicad_pcb (KiCad board)
At the start: 2 copper layers, 300 x 114.3 mm, 185 parts, among them J1 JST SH, J2 Pico EZmate, SW1 RotaryEncoder_Switch, SW2 RotaryEncoder_Switch, SW3 RotaryEncoder_Switch, SW4 RotaryEncoder_Switch, SW5 SKQGABE010, U1 XC6206PxxxMR-Regulator_Linear, U2 STM32F072CBT6

Commit message: silkscreen correction, fresh gerbers
Other:
- board text added: "HP2621"
- board text removed: "HP2612"
Changed lines of the file:
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@@
     (fp_arc (start 8.53125 -5.499999) (mid 8.677685 -5.853565) (end 9.03125 -5.999999)
       (stroke (width 0.05) (type solid)) (layer "Eco2.User"))
-    (fp_arc (start 9.03125 8.000001) (mid 8.677729 7.853537) (end 8.53125 7.500001)
+    (fp_arc (start 9.03125 8.000001) (mid 8.677693 7.853543) (end 8.53125 7.500001)
       (stroke (width 0.05) (type solid)) (layer "Eco2.User"))
-    (fp_arc (start 14.780039 -5.999999) (mid 15.133567 -5.853539) (end 15.280039 -5.499999)
+    (fp_arc (start 14.780039 -5.999999) (mid 15.133602 -5.853545) (end 15.280039 -5.499999)
       (stroke (width 0.05) (type solid)) (layer "Eco2.User"))
-    (fp_arc (start 15.28125 7.500001) (mid 15.134806 7.853571) (end 14.78125 8.000001)
+    (fp_arc (start 15.28125 7.500001) (mid 15.1348 7.853536) (end 14.78125 8.000001)
       (stroke (width 0.05) (type solid)) (layer "Eco2.User"))
     (fp_circle (center -11.90625 -6.985) (end -9.90625 -6.985)
@@
     (effects (font (size 0.9 0.9) (thickness 0.15)) (justify mirror))
   )
-  (gr_text "HP2612" (at 261.9375 116.68125) (layer "B.SilkS")
+  (gr_text "HP2621" (at 261.9375 116.68125) (layer "B.SilkS")
     (effects (font (size 4 4) (thickness 0.6) bold) (justify mirror))
   )
@@
     (effects (font (size 0.9 0.9) (thickness 0.15)) (justify mirror))
   )
-  (gr_text "HP2612" (at 270.66875 119.85625) (layer "F.SilkS")
+  (gr_text "HP2621" (at 270.66875 119.85625) (layer "F.SilkS")
     (effects (font (size 6 6) (thickness 0.6) bold))
   )

Commit message: fresh gerbers
Routing:
- net COL7: track 270.2 -> 272.2 mm
- net ENC_g: track 140.0 -> 141.6 mm
- net ROW4: track 318.8 -> 320.0 mm
- net COL1: track 126.5 -> 127.5 mm
- net COL4: track 227.8 -> 228.6 mm
- net COL5: track 264.5 -> 265.4 mm
- net COL3: track 231.3 -> 232.0 mm
- net ROW5: track 290.0 -> 290.7 mm
- net COL2: track 207.3 -> 208.0 mm
- net COL6: track 230.5 -> 231.1 mm
- net ENC_h: track 137.0 -> 137.6 mm
